File: hardware/kicad/stevekey/stevekey.kicad_pcb (KiCad board)
At the start: 2 copper layers, 60.4 x 49.1 mm, 24 parts, among them J1 ATMEL-ICE-10, J2 Conn_01x04, J3 Conn_01x02, J4 Conn_01x02, J5 Conn_01x02, Q1 2N3904, SW1 SW_SL, SW2 SW_CAPS, SW3 SW_4080, U1 CD4066BM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

Commit message: Use internal pull-ups for keys
Parts:
- removed R1, R2, R3: 10K, Resistor_THT:R_Axial_DIN0204_L3.6mm_D1.6mm_P7.62mm_Horizontal
- J2: value Conn_01x04 -> Conn_01x06
- R4, R5, R6: value 150 -> 330
- U2: value ATtiny214-SS -> ATtiny214/414/814
Routing:
- net N4080KEY: track 60.7 -> 47.2 mm
- net NCAPSKEY: track 47.5 -> 34.8 mm
- net VCC: track 138.2 -> 145.2 mm
- net NSLKEY: track 39.9 -> 38.9 mm, vias 1 -> 2
Other:
- board text added: "STEVEKEY MCU DEV BOARD REV. 2 © 2023 MIKE NABEREZNY"
- board text added: "▲ ATTINY414"
- board text removed: "STEVEKEY MCU DEV BOARD REV. 1 © 2023 MIKE NABEREZNY"
- board text removed: "▲ ATTINY214"
